Commit message: feat: unify robot control safety stack and add web GUI

File: software/leap_ros_ws/src/xuegecar_description/urdf/xuegecar.urdf (robot description, URDF)
Before this commit: robot xuegecar, 7 links, 6 joints
Links:
- link base_link: geometry collision box size=0.1565 0.145 0.145; visual box size=0.1565 0.145 0.145
- link imu_link: geometry visual box size=0.02 0.02 0.01
- link laser_frame: geometry visual cylinder length=0.014 radius=0.02
- link left_wheel_link: geometry visual cylinder length=0.04 radius=0.0325
- link right_wheel_link: geometry visual cylinder length=0.04 radius=0.0325
Joints:
- joint base_joint: origin xyz=0.0 0.0 0.076 rpy=0 0 0 -> xyz=0 0 0.0325 rpy=0 0 0
- joint caster_joint: axis 0 1 0 -> (none); origin xyz=0.06 0.0 -0.076 -> xyz=0.080 0 -0.0165 rpy=0 0 0
- joint imu_joint: origin xyz=0 0 0.02 -> xyz=0.020 0 0.0635 rpy=0 0 0
- joint laser_joint: origin xyz=0 0 0.075 -> xyz=0.020 0 0.1055 rpy=0 0 0
- joint left_wheel_joint: origin xyz=-0.02 0.10 -0.06 -> xyz=0 0.0525 0 rpy=0 0 0
- joint right_wheel_joint: origin xyz=-0.02 -0.10 -0.06 -> xyz=0 -0.0525 0 rpy=0 0 0
